Commit message: Update master urdf for reachability search.

File: stl2urdf/assets/Assem_4310_JOINT/Assem_4310_JOINT/urdf/Assem_4310_JOINT.urdf (robot description, URDF)
Before this commit: robot Assem_4310_JOINT, 2 links, 1 joints
Joints:
- joint motor4310_rev_joint: origin xyz=0.0255 -0.0395 0 rpy=0 0 0 -> xyz=0.0255 -0.0395 0 rpy=0 0 1.57
