Commit message: fixed rotational issues with 540_joint and added correct version of 540_base

File: ga/assets/540_base/540_base/urdf/540_base.urdf (robot description, URDF)
Before this commit: robot 540_base, 2 links, 1 joints
Links:
- removed link adaptor_link
- added link joint1, mass 0.016459; collision mesh filename=package://540_base/meshes/joint1.STL; visual mesh filename=package://540_base/meshes/joint1.STL
- link base_link: mass 0.177193779086753 -> 0.182418164745937
Joints:
- removed joint adaptor_joint
- added joint joint1: type continuous, parent base_link, child joint1, origin xyz=0.016 0 0.0575 rpy=0 0 -0.17953295, axis 0 0 1
