Commit message: ga pipeline with updated modules

File: ga/robot6DOF.urdf (robot description, URDF)
Before this commit: robot Auto-Generated: 0dd55ee4e9004159aa950d384653e475, 18 links, 17 joints
Links:
- removed link motor4305_rev_joint.motor4305_link
- removed link motor4305_rev_joint.motor4305_out_link
- removed link motor4305_rev_joint.motor4305_out_link.motor4305_out_linkconnector.body
- removed link r4310to4305-0.15.r4310to4305-0.15
- added link eef.EEF, mass 0.0; collision sphere radius=0.02; visual sphere radius=0.02
- added link eef.EEF.end-effector.body
- added link motor4310_rev_joint-4.motor4310_in_link, mass 0.57649; collision mesh filename=assets/Assem_4310_JOINT/Assem_4310_JOINT/meshes/motor4310_i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 scale=1.0 1.0 1.0; visual mesh filename=assets/Assem_4310_JOINT/Assem_4310_JOINT/meshes/motor4310_i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 scale=1.0 1.0 1.0
- added link motor4310_rev_joint-4.motor4310_out_link, mass 0.088545; collision mesh filename=assets/Assem_4310_JOINT/Assem_4310_JOINT/meshes/motor4310_o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 scale=1.0 1.0 1.0; visual mesh filename=assets/Assem_4310_JOINT/Assem_4310_JOINT/meshes/motor4310_o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 scale=1.0 1.0 1.0
- added link r4310to4310-0.3.r4310to4310-0.3, mass 0.00018750000000000003; collision box size=0.025 0.025 0.3; visual box size=0.025 0.025 0.3
- added link r4310to4310-0.45.r4310to4310-0.45, mass 0.0002812500000000001; collision box size=0.025 0.025 0.45; visual box size=0.025 0.025 0.45
Joints:
- removed joint motor4305_rev_joint.motor4305_link.motor4305_linkconnector
- removed joint motor4305_rev_joint.motor4305_out_link.motor4305_out_linkconnector
- removed joint motor4305_rev_joint.motor4305_rev_joint
- removed joint r4310to4305-0.15.r4310to4305-0.15.2-1
- added joint eef.EEF.end-effector: type fixed, parent eef.EEF, child eef.EEF.end-effector.body, origin xyz=0.0 0.02666666666667 0.0 rpy=3.141592653589793 0.0 0.0
- added joint eef.EEF.robot2eef: type fixed, parent r4310to4310-0.15-2.r4310to4310-0.15, child eef.EEF, origin xyz=0.0 0.025 0.125 rpy=-1.5707963267948966 0.0 -3.141592653589793
- added joint motor4310_rev_joint-4.motor4310_in_link.motor4310_in_linkconnector: type fixed, parent r4310to4310-0.15-1.r4310to4310-0.15, child motor4310_rev_joint-4.motor4310_in_link, origin xyz=0.0 0.025 0.125 rpy=-1.5707963267948966 0.0 -3.141592653589793
- added joint motor4310_rev_joint-4.motor4310_rev_joint: type revolute, parent motor4310_rev_joint-4.motor4310_in_link, child motor4310_rev_joint-4.motor4310_out_link, origin xyz=0.02549999999838 -0.03949999999748 0.0 rpy=1.5707963267948966 0.0 1.56999999997889, axis 0 0 1, limit lower=-3.141592653589793 upper=3.141592653589793 effort=1000.0 velocity=10.0
- added joint r4310to4310-0.3.r4310to4310-0.3.2-1: type fixed, parent motor4310_rev_joint-2.motor4310_out_link, child r4310to4310-0.3.r4310to4310-0.3, origin xyz=0.0 0.0 0.0 rpy=1.5707963267948966 0.0 0.0
- added joint r4310to4310-0.45.r4310to4310-0.45.2-1: type fixed, parent motor4310_rev_joint.motor4310_out_link, child r4310to4310-0.45.r4310to4310-0.45, origin xyz=0.0 0.0 0.0 rpy=1.5707963267948966 0.0 0.0
- joint motor4310_rev_joint-1.motor4310_in_link.motor4310_in_linkconnector: origin xyz=0.0 0.025 0.125 rpy=-1.5707963267948966 0.0 -3.141592653589793 -> xyz=0.0 0.025 0.425 rpy=-1.5707963267948966 0.0 -3.141592653589793; parent r4310to4310-0.15.r4310to4310-0.15 -> r4310to4310-0.45.r4310to4310-0.45
- joint motor4310_rev_joint-2.motor4310_in_link.motor4310_in_linkconnector: parent r4310to4310-0.15-1.r4310to4310-0.15 -> r4310to4310-0.15.r4310to4310-0.15
- joint motor4310_rev_joint-3.motor4310_in_link.motor4310_in_linkconnector: origin xyz=0.0 0.025 0.125 rpy=-1.5707963267948966 0.0 -3.141592653589793 -> xyz=0.0 0.025 0.275 rpy=-1.5707963267948966 0.0 -3.141592653589793; parent r4310to4310-0.15-2.r4310to4310-0.15 -> r4310to4310-0.3.r4310to4310-0.3
- joint r4310to4310-0.15-1.r4310to4310-0.15.2-1: parent motor4310_rev_joint-1.motor4310_out_link -> motor4310_rev_joint-3.motor4310_out_link
- joint r4310to4310-0.15-2.r4310to4310-0.15.2-1: parent motor4310_rev_joint-2.motor4310_out_link -> motor4310_rev_joint-4.motor4310_out_link
- joint r4310to4310-0.15.r4310to4310-0.15.2-1: parent motor4310_rev_joint.motor4310_out_link -> motor4310_rev_joint-1.motor4310_out_link

Commit message: added optimal solution urdf

File: ga/robot6DOF.urdf (robot description, URDF)
Before this commit: robot Auto-Generated: 3ccd00c199ff4cfd81bc3fa710332e28, 20 links, 19 joints
Links:
- removed link base_rev_joint.base_motor_link
- removed link base_rev_joint.base_out_link
- removed link baseto4310-0.15.baseto4310-0.15
- removed link motor4310_rev_joint-1.motor4310_in_link
- removed link motor4310_rev_joint-1.motor4310_out_link
- removed link motor4310_rev_joint-2.motor4310_in_link
- removed link motor4310_rev_joint-2.motor4310_out_link
- removed link motor4310_rev_joint-3.motor4310_in_link
- removed link motor4310_rev_joint-3.motor4310_out_link
- removed link motor4310_rev_joint-4.motor4310_in_link
- removed link motor4310_rev_joint-4.motor4310_out_link
- removed link motor4310_rev_joint.motor4310_in_link
- removed link motor4310_rev_joint.motor4310_out_link
- removed link r4310to4310-0.15-1.r4310to4310-0.15
- removed link r4310to4310-0.15-2.r4310to4310-0.15
- removed link r4310to4310-0.15.r4310to4310-0.15
- removed link r4310to4310-0.3.r4310to4310-0.3
- removed link r4310to4310-0.45.r4310to4310-0.45
- added link 330_joint-1.330_jointAdaptor_Link, mass 0.0172446569319253; collision mesh filename=assets/330_joint/330_joint/meshes/Adaptor_Link.STL scale=1.0 1.0 1.0; visual mesh filename=assets/330_joint/330_joint/meshes/Adaptor_Link.STL scale=1.0 1.0 1.0
- added link 330_joint-1.330_jointbase_link, mass 0.044407; collision mesh filename=assets/330_joint/330_joint/meshes/base_link.STL scale=1.0 1.0 1.0; visual mesh filename=assets/330_joint/330_joint/meshes/base_link.STL scale=1.0 1.0 1.0
- added link 330_joint-to-430_joint-0.2-0-N.330_joint-to-430_joint-0.2-0-N, mass 0.00012500000000000003; collision box size=0.025 0.025 0.2; visual box size=0.025 0.025 0.2
- added link 330_joint-to-540_joint-0.1-3-W.330_joint-to-540_joint-0.1-3-W, mass 6.250000000000001e-05; collision box size=0.025 0.025 0.1; visual box size=0.025 0.025 0.1
- added link 330_joint.330_jointAdaptor_Link, mass 0.0172446569319253; collision mesh filename=assets/330_joint/330_joint/meshes/Adaptor_Link.STL scale=1.0 1.0 1.0; visual mesh filename=assets/330_joint/330_joint/meshes/Adaptor_Link.STL scale=1.0 1.0 1.0
- added link 330_joint.330_jointbase_link, mass 0.044407; collision mesh filename=assets/330_joint/330_joint/meshes/base_link.STL scale=1.0 1.0 1.0; visual mesh filename=assets/330_joint/330_joint/meshes/base_link.STL scale=1.0 1.0 1.0
- added link 430_joint-to-540_joint-0.15-0-W.430_joint-to-540_joint-0.15-0-W, mass 9.375000000000002e-05; collision box size=0.025 0.025 0.15; visual box size=0.025 0.025 0.15
- added link 430_joint.430_jointadaptor_Link, mass 0.0139178998268077; collision mesh filename=assets/430_joint/430_joint/meshes/adaptor_Link.STL scale=1.0 1.0 1.0; visual mesh filename=assets/430_joint/430_joint/meshes/adaptor_Link.STL scale=1.0 1.0 1.0
- added link 430_joint.430_jointbase_link, mass 0.0706732385140066; collision mesh filename=assets/430_joint/430_joint/meshes/base_link.STL scale=1.0 1.0 1.0; visual mesh filename=assets/430_joint/430_joint/meshes/base_link.STL scale=1.0 1.0 1.0
- added link 540_base-to-330_joint-0.1-1-S.540_base-to-330_joint-0.1-1-S, mass 6.250000000000001e-05; collision box size=0.025 0.025 0.1; visual box size=0.025 0.025 0.1
- added link 540_base.540_basebase_link, mass 0.182418164745937; collision mesh filename=assets/540_base/540_base/meshes/base_link.STL scale=1.0 1.0 1.0; visual mesh filename=assets/540_base/540_base/meshes/base_link.STL scale=1.0 1.0 1.0
- added link 540_base.540_basejoint1, mass 0.016459; collision mesh filename=assets/540_base/540_base/meshes/joint1.STL scale=1.0 1.0 1.0; visual mesh filename=assets/540_base/540_base/meshes/joint1.STL scale=1.0 1.0 1.0
- added link 540_joint-1.540_jointadaptor_link, mass 0.0164593396501985; collision mesh filename=assets/540_joint/540_joint/meshes/adaptor_link.STL scale=1.0 1.0 1.0; visual mesh filename=assets/540_joint/540_joint/meshes/adaptor_link.STL scale=1.0 1.0 1.0
- added link 540_joint-1.540_jointbase_link, mass 0.125294353341299; collision mesh filename=assets/540_joint/540_joint/meshes/base_link.STL scale=1.0 1.0 1.0; visual mesh filename=assets/540_joint/540_joint/meshes/base_link.STL scale=1.0 1.0 1.0
- added link 540_joint-to-330_joint-0.2-1-E.540_joint-to-330_joint-0.2-1-E, mass 0.00012500000000000003; collision box size=0.025 0.025 0.2; visual box size=0.025 0.025 0.2
- added link 540_joint-to-430_joint-0.3-0-E.540_joint-to-430_joint-0.3-0-E, mass 0.00018750000000000003; collision box size=0.025 0.025 0.3; visual box size=0.025 0.025 0.3
- added link 540_joint.540_jointadaptor_link, mass 0.0164593396501985; collision mesh filename=assets/540_joint/540_joint/meshes/adaptor_link.STL scale=1.0 1.0 1.0; visual mesh filename=assets/540_joint/540_joint/meshes/adaptor_link.STL scale=1.0 1.0 1.0
- added link 540_joint.540_jointbase_link, mass 0.125294353341299; collision mesh filename=assets/540_joint/540_joint/meshes/base_link.STL scale=1.0 1.0 1.0; visual mesh filename=assets/540_joint/540_joint/meshes/base_link.STL scale=1.0 1.0 1.0
- link eef.EEF: geometry collision sphere radius=0.013333333333333334; visual sphere radius=0.013333333333333334
Joints:
- removed joint base_rev_joint.base_rev_joint
- removed joint baseto4310-0.15.baseto4310-0.15.2-1
- removed joint motor4310_rev_joint-1.motor4310_in_link.motor4310_in_linkconnector
- removed joint motor4310_rev_joint-1.motor4310_rev_joint
- removed joint motor4310_rev_joint-2.motor4310_in_link.motor4310_in_linkconnector
- removed joint motor4310_rev_joint-2.motor4310_rev_joint
- removed joint motor4310_rev_joint-3.motor4310_in_link.motor4310_in_linkconnector
- removed joint motor4310_rev_joint-3.motor4310_rev_joint
- removed joint motor4310_rev_joint-4.motor4310_in_link.motor4310_in_linkconnector
- removed joint motor4310_rev_joint-4.motor4310_rev_joint
- removed joint motor4310_rev_joint.motor4310_in_link.motor4310_in_linkconnector
- removed joint motor4310_rev_joint.motor4310_rev_joint
- removed joint r4310to4310-0.15-1.r4310to4310-0.15.2-1
- removed joint r4310to4310-0.15-2.r4310to4310-0.15.2-1
- removed joint r4310to4310-0.15.r4310to4310-0.15.2-1
- removed joint r4310to4310-0.3.r4310to4310-0.3.2-1
- removed joint r4310to4310-0.45.r4310to4310-0.45.2-1
- added joint 330_joint-1.330_joint: type revolute, parent 330_joint-1.330_jointbase_link, child 330_joint-1.330_jointAdaptor_Link, origin xyz=0.0201 -0.0147 0.0246 rpy=-1.5707963267948966 0.0 -3.141592653589793, axis 0 0 1, limit lower=-inf upper=inf effort=1000.0 velocity=10.0
- added joint 330_joint-1.330_jointbase_link.330_jointbase_linkconnector: type fixed, parent 540_joint-to-330_joint-0.2-1-E.540_joint-to-330_joint-0.2-1-E, child 330_joint-1.330_jointbase_link, origin xyz=-0.0125 0.2425 -0.03 rpy=1.5707963267949068 0.0 -1.5707963267948966
- added joint 330_joint-to-430_joint-0.2-0-N.330_joint-to-430_joint-0.2-0-N.2-1: type fixed, parent 330_joint-1.330_jointAdaptor_Link, child 330_joint-to-430_joint-0.2-0-N.330_joint-to-430_joint-0.2-0-N, origin xyz=0.0 0.0 0.0 rpy=3.141592653589793 0.0 0.0
- added joint 330_joint-to-540_joint-0.1-3-W.330_joint-to-540_joint-0.1-3-W.2-1: type fixed, parent 330_joint.330_jointAdaptor_Link, child 330_joint-to-540_joint-0.1-3-W.330_joint-to-540_joint-0.1-3-W, origin xyz=0.0 0.0 0.0 rpy=3.141592653589793 0.0 0.0
- added joint 330_joint.330_joint: type revolute, parent 330_joint.330_jointbase_link, child 330_joint.330_jointAdaptor_Link, origin xyz=0.0201 -0.0147 0.0246 rpy=-1.5707963267948966 0.0 -3.141592653589793, axis 0 0 1, limit lower=-inf upper=inf effort=1000.0 velocity=10.0
- added joint 330_joint.330_jointbase_link.330_jointbase_linkconnector: type fixed, parent 540_base-to-330_joint-0.1-1-S.540_base-to-330_joint-0.1-1-S, child 330_joint.330_jointbase_link, origin xyz=-0.00217060222084 -0.01231009691265 -0.1175 rpy=1.3962634015954656 -1.5707963267948966 0.0
- added joint 430_joint-to-540_joint-0.15-0-W.430_joint-to-540_joint-0.15-0-W.2-1: type fixed, parent 430_joint.430_jointadaptor_Link, child 430_joint-to-540_joint-0.15-0-W.430_joint-to-540_joint-0.15-0-W, origin xyz=0.0 0.0 0.0 rpy=3.141592653589793 0.0 0.0
- added joint 430_joint.430_joint: type revolute, parent 430_joint.430_jointbase_link, child 430_joint.430_jointadaptor_Link, origin xyz=0.0 0.0011 -0.0 rpy=1.5707963267948966 0.0 0.0, axis 0 0 1, limit lower=-inf upper=inf effort=1000.0 velocity=10.0
- added joint 430_joint.430_jointbase_link.430_jointbase_linkconnector: type fixed, parent 540_joint-to-430_joint-0.3-0-E.540_joint-to-430_joint-0.3-0-E, child 430_joint.430_jointbase_link, origin xyz=0.0 0.39875 -0.04875 rpy=1.5707963267948966 9.992007221626409e-15 3.141592653589793
- added joint 540_base-to-330_joint-0.1-1-S.540_base-to-330_joint-0.1-1-S.2-1: type fixed, parent 540_base.540_basejoint1, child 540_base-to-330_joint-0.1-1-S.540_base-to-330_joint-0.1-1-S, origin xyz=0.0 0.0 0.0 rpy=3.141592653589793 0.0 0.0
- added joint 540_base.540_base: type revolute, parent 540_base.540_basebase_link, child 540_base.540_basejoint1, origin xyz=0.016 0.0 0.0575 rpy=0.0 0.0 -0.17953294999999775, axis 0 0 1, limit lower=-inf upper=inf effort=1000.0 velocity=10.0
- added joint 540_joint-1.540_joint: type revolute, parent 540_joint-1.540_jointbase_link, child 540_joint-1.540_jointadaptor_link, origin xyz=0.0 0.0 0.03 rpy=1.5707963267948966 0.0 0.0, axis 0 0 1, limit lower=-inf upper=inf effort=1000.0 velocity=10.0
- added joint 540_joint-1.540_jointbase_link.540_jointbase_linkconnector: type fixed, parent 430_joint-to-540_joint-0.15-0-W.430_joint-to-540_joint-0.15-0-W, child 540_joint-1.540_jointbase_link, origin xyz=0.0 0.0 -0.185 rpy=-3.141592653589793 0.0 -3.1415926535897833
- added joint 540_joint-to-330_joint-0.2-1-E.540_joint-to-330_joint-0.2-1-E.2-1: type fixed, parent 540_joint-1.540_jointadaptor_link, child 540_joint-to-330_joint-0.2-1-E.540_joint-to-330_joint-0.2-1-E, origin xyz=0.0 -0.03 0.0 rpy=1.5707963267948966 0.0 0.0
- added joint 540_joint-to-430_joint-0.3-0-E.540_joint-to-430_joint-0.3-0-E.2-1: type fixed, parent 540_joint.540_jointadaptor_link, child 540_joint-to-430_joint-0.3-0-E.540_joint-to-430_joint-0.3-0-E, origin xyz=0.0 -0.03 0.0 rpy=1.5707963267948966 0.0 0.0
- added joint 540_joint.540_joint: type revolute, parent 540_joint.540_jointbase_link, child 540_joint.540_jointadaptor_link, origin xyz=0.0 0.0 0.03 rpy=1.5707963267948966 0.0 0.0, axis 0 0 1, limit lower=-inf upper=inf effort=1000.0 velocity=10.0
- added joint 540_joint.540_jointbase_link.540_jointbase_linkconnector: type fixed, parent 330_joint-to-540_joint-0.1-3-W.330_joint-to-540_joint-0.1-3-W, child 540_joint.540_jointbase_link, origin xyz=0.0 0.0792038367717 -0.0625 rpy=3.141592653589793 0.0 3.141592653589793
- joint eef.EEF.robot2eef: origin xyz=0.0 0.025 0.125 rpy=-1.5707963267948966 0.0 -3.141592653589793 -> xyz=0.0 -0.01875 -0.2604538367717 rpy=3.141592653589793 0.0 3.141592653589793; parent r4310to4310-0.15-2.r4310to4310-0.15 -> 330_joint-to-430_joint-0.2-0-N.330_joint-to-430_joint-0.2-0-N
