Commit message: added some options to simplify db

File: ga/assets/330_joint/330_joint/urdf/330_joint.urdf (robot description, URDF)
Before this commit: robot 330_joint, 2 links, 1 joints
Links:
- link base_link: mass 0.044407 -> 0.067407

File: ga/assets/430_joint/430_joint/urdf/430_joint.urdf (robot description, URDF)
Before this commit: robot 430_joint, 2 links, 1 joints
Links:
- link base_link: mass 0.0706732385140066 -> 0.15267323851

File: ga/assets/540_base/540_base/urdf/540_base.urdf (robot description, URDF)
Before this commit: robot 540_base, 2 links, 1 joints
Links:
- link base_link: mass 0.182418164745937 -> 0.35041816474

File: ga/assets/540_joint/540_joint/urdf/540_joint.zip.urdf (robot description, URDF)
Before this commit: robot 540_joint.zip, 2 links, 1 joints
Links:
- link base_link: mass 0.125294353341299 -> 0.29029435334
